File: ESP32chat.kicad_sch (KiCad schematic)
At the start: 112 parts, among them J1 CONN_021X02_NO_SILK, J2 CONN_021X02_NO_SILK, J3 CONN_01, Q1 Si1308, Q2 BSS123, U1 tp4056_KoreanHropartsElecTYPE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, U2 RFM69HCW, U3 ESP32, U4 BUZZER, U5 FPCConn, U6 RT9013, U7 MCP73831T-2ACI/OT, X1 uFL

Commit message: DRAFT Still needs silk screen, would be nice to remove errors.
Parts:
- renumbered U$3 to U10, U$4 to U11, U$5 to U12, U$6 to U13, U$7 to U14, U$8 to U15, U$1 to U8, U$2 to U9
Connections:
- net EPD_MISO is gone; now on net LORA_MISO: U3.34 (MTDI/GPIO41/CLK_OUT1)
- net IO43 is gone; now on net LORA_CS: U3.37 (U0TXD/GPIO43/CLK_OUT1)
- net IO44 is gone; now on net LORA_SCK: U3.36 (U0RXD/GPIO44/CLK_OUT2)
- net COL01: now also U3.9 (GPIO16/U0CTS/ADC2_CH5/XTAL_32K_NH5); no longer U3.6 (GPIO6/TOUCH6/ADC1_CH5)
- net COL02: now also U3.10 (GPIO17/U1TXD/ADC2_CH6); no longer U3.4 (GPIO4/TOUCH4/ADC1_CH3)
- net COL03: now also U3.11 (GPIO18/U1RXD/ADC2_CH7/CLK_OUT3); no longer U3.7 (GPIO7/TOUCH7/ADC1_CH6)
- net COL04: now also U3.12 (GPIO8/TOUCH8/ADC1_CH7/SUBSPICS1); no longer U3.19 (GPIO11/TOUCH11/ADC2_CH0/FSPICS0/FSPIIO4/SUBSPICS0)
- net COL05: now also U3.15 (GPIO3/TOUCH3/ADC1_CH2); no longer U3.20 (GPIO12/TOUCH11/ADC2_CH0/FSPICS0/FSPIIO4/SUBSPICS0)
- net COL06: now also U3.16 (GPIO46); no longer U3.21 (GPIO13/TOUCH13/ADC2_CH2/FSPIQ/FSPIIO7/SUBSPIQ)
- net COL07: now also U3.17 (GPIO9/TOUCH9/ADC1_CH8/FSPIHD/SUBSPIHD); no longer U3.22 (GPIO14/TOUCH14/ADC2_CH3/FSPIWP/FSPIDQS/SUBSPIWP)
- net COL08: now also U3.18 (GPIO10/TOUCH10/ADC1_CH9/FSPICS0/FSPIIO4/SUBSPICS0); no longer U3.10 (GPIO17/U1TXD/ADC2_CH6)
- net COL09: now also U3.19 (GPIO11/TOUCH11/ADC2_CH0/FSPICS0/FSPIIO4/SUBSPICS0); no longer U3.11 (GPIO18/U1RXD/ADC2_CH7/CLK_OUT3)
- net COL10: now also U3.20 (GPIO12/TOUCH11/ADC2_CH0/FSPICS0/FSPIIO4/SUBSPICS0); no longer U3.38 (GPIO2/TOUCH2/ADC1_CH1), U3.39 (GPIO1/TOUCH1/ADC1_CH0)
- net COL11: now also U3.21 (GPIO13/TOUCH13/ADC2_CH2/FSPIQ/FSPIIO7/SUBSPIQ); no longer U3.15 (GPIO3/TOUCH3/ADC1_CH2)
- net EPD_BUSY: now also U3.32 (MTCK/GPIO39/CLK_OUT3/SUBSPICS1); no longer U3.28 (SPIIO6/GPIO35/FSPID/SUBSPID)
- net EPD_CLK: now also U3.28 (SPIIO6/GPIO35/FSPID/SUBSPID); no longer U3.33 (MTDO/GPIO40/CLK_OUT2)
- net EPD_CS: now also U3.29 (SPIIO7/GPIO36/FSPICLK/SUBSPICLK); no longer U3.32 (MTCK/GPIO39/CLK_OUT3/SUBSPICS1)
- net EPD_MOSI: now also U3.26 (GPIO45); no longer U3.35 (MTMS/GPIO42)
- net EPD_RST: now also U3.31 (GPIO38/FSPIWP/SUBSPIWP); no longer U3.29 (SPIIO7/GPIO36/FSPICLK/SUBSPICLK)
- net LORA_IRQ: now also U3.39 (GPIO1/TOUCH1/ADC1_CH0); no longer U3.24 (GPIO47/SPICLK_P/SUBSPICLK_P_DIFF)
- net LORA_MISO: no longer U3.26 (GPIO45)
- net LORA_MOSI: now also U3.35 (MTMS/GPIO42); no longer U3.23 (GPIO21)
- net LORA_RST: now also U3.38 (GPIO2/TOUCH2/ADC1_CH1); no longer U3.25 (GPIO48/SPICLK_N/SUBSPICLK_N_DIFF)
- net LORA_SCK: no longer U3.16 (GPIO46)
- net ROW01: now also U3.22 (GPIO14/TOUCH14/ADC2_CH3/FSPIWP/FSPIDQS/SUBSPIWP)
- net ROW02: now also U3.23 (GPIO21); no longer U3.5 (GPIO5/TOUCH5/ADC1_CH4)
- net ROW03: now also U3.24 (GPIO47/SPICLK_P/SUBSPICLK_P_DIFF); no longer U3.17 (GPIO9/TOUCH9/ADC1_CH8/FSPIHD/SUBSPIHD)
- net ROW04: now also U3.25 (GPIO48/SPICLK_N/SUBSPICLK_N_DIFF); no longer U3.18 (GPIO10/TOUCH10/ADC1_CH9/FSPICS0/FSPIIO4/SUBSPICS0)
- net RXLED: now also U3.5 (GPIO5/TOUCH5/ADC1_CH4); no longer U3.12 (GPIO8/TOUCH8/ADC1_CH7/SUBSPICS1)
- net SPEAKPWM: now also U3.33 (MTDO/GPIO40/CLK_OUT2); no longer U3.31 (GPIO38/FSPIWP/SUBSPIWP)
- net TXLED: now also U3.4 (GPIO4/TOUCH4/ADC1_CH3); no longer U3.9 (GPIO16/U0CTS/ADC2_CH5/XTAL_32K_NH5)
- net ROW1 renamed IO15
- new net IO06: U3.6 (GPIO6/TOUCH6/ADC1_CH5)
- new net IO07: U3.7 (GPIO7/TOUCH7/ADC1_CH6)
- no-connect marks 12 -> 19

Commit message: Almost ready for review.
Parts:
- BT1: JLCPCB C2988620 -> (none); LCSC (none) -> C2988620
- C1, C5: value 1U -> 1u; LCSC (none) -> C15849
- C10, C11, C13, C14, C15, C16, C3, C4, C8, C9: LCSC (none) -> C15849
- C12: LCSC (none) -> C194427
- C17, C19, C21, C22: value 10µF -> 10u; LCSC (none) -> C194427
- C18, C6: LCSC (none) -> C14663
- C2: value 10uF -> 10u; LCSC (none) -> C194427
- C20, C23: value 1µF -> 1u; LCSC (none) -> C15849
- C7: LCSC (none) -> C162274
- D1, D2, D3: LCSC (none) -> C77336
- GRN1: LCSC (none) -> C434432
- J1, J2, J3, JP1, LOGO2, U10, U11, U12, U13, U14, U15, U8, U9: LCSC (none) -> DNP
- L1: JLCPCB C9393 -> (none); LCSC (none) -> C9393
- LOGO1: JLCPCB C108781 -> (none); LCSC (none) -> C108781
- ORG1: LCSC (none) -> C84262
- Q1: JLCPCB C469327 -> (none); LCSC (none) -> C469327
- Q2: LCSC (none) -> C79015
- R1, R2: LCSC (none) -> C22843
- R10: LCSC (none) -> C23411
- R11, R13, R7, R8, R9: LCSC (none) -> C25804
- R12, R6: LCSC (none) -> C21190
- R3: value 5.1K -> 5K1; LCSC (none) -> C23186
- R4, R5: LCSC (none) -> C21189
- RED1: LCSC (none) -> C84256
- S1, S10, S11, S12, S13, S14, S15, S16, S17, S18, S19, S2, S20, S21, S22, S23, S24, S25, S26, S27, S28, S29, S3, S30, S31, S32, S33, S34, S35, S36, S37, S38, S39, S4, S40, S41, S42, S43, S44, S5, S6, S7, S8, S9: JLCPCB C318886 -> (none); LCSC (none) -> C318886
- U1: JLCPCB C134092 -> (none); LCSC (none) -> C134092
- U2: JLCPCB C2844473 -> (none); LCSC (none) -> C2844473
- U3: JLCPCB C2913199 -> (none); LCSC (none) -> C2913199
- U4: JLCPCB C482342 -> (none); LCSC (none) -> C482342
- U5: JLCPCB C11092 -> (none); LCSC (none) -> C11092
- U6: LCSC (none) -> C47773
- U7: JLCPCB C424093 -> (none); LCSC (none) -> C424093
- X1: JLCPCB C411575 -> (none); LCSC (none) -> C411575

Commit message: DRAFT added solar charging circuit, changed to 6X6 key scanning, 36 buttons with less consumed GPIO. Added temperature sensor to monitor the battery. Added GPS module.
Parts:
- removed C17: 10u, Capacitor_SMD:C_0603_1608Metric, symbol Device:C_Small
- removed S11: BSP, KICAD_Footprints:TS-1187A-C-G-B, symbol Switch:SW_Push
- removed S18: U, KICAD_Footprints:TS-1187A-C-G-B, symbol Switch:SW_Push
- removed S22: ENT, KICAD_Footprints:TS-1187A-C-G-B, symbol Switch:SW_Push
- removed S29: J, KICAD_Footprints:TS-1187A-C-G-B, symbol Switch:SW_Push
- removed S33: _, KICAD_Footprints:TS-1187A-C-G-B, symbol Switch:SW_Push
- removed S40: M, KICAD_Footprints:TS-1187A-C-G-B, symbol Switch:SW_Push
- removed S44: >, KICAD_Footprints:TS-1187A-C-G-B, symbol Switch:SW_Push
- removed S7: 7, KICAD_Footprints:TS-1187A-C-G-B, symbol Switch:SW_Push
- added AE1: Antenna_Shield, Connector_Coaxial:U.FL_Hirose_U.FL-R-SMT-1_Vertical, symbol Device:Antenna_Shield
- added C1, C8: 10u, Capacitor_SMD:C_0603_1608Metric, symbol Device:C
- added C6, C9: 100n, Capacitor_SMD:C_0603_1608Metric, symbol Device:C
- added D1: MBR0530, Diode_SMD:D_SOD-123, symbol Diode:MBR0530
- added GRN2: GRN, LED_SMD:LED_0805_2012Metric, symbol Device:LED
- added J1, J3: CONN_021X02_NO_SILK, Connector_PinHeader_2.54mm:PinHeader_1x02_P2.54mm_Vertical, symbol Connector_Generic:Conn_01x02
- added L1: 6.8nH, Inductor_SMD:L_0603_1608Metric, symbol Device:L
- added Q1: Q_PMOS_DGS, Package_TO_SOT_SMD:SOT-23, symbol Device:Q_PMOS_DGS
- added R10, R16: 10K, Resistor_SMD:R_0603_1608Metric, symbol Device:R
- added R11, R14, R15: 1K, Resistor_SMD:R_0603_1608Metric, symbol Device:R
- added R12, R13: 50K, Resistor_SMD:R_0603_1608Metric, symbol Device:R
- added R17: 0R, Resistor_SMD:R_0603_1608Metric, symbol Device:R
- added R9: 100, Resistor_SMD:R_0603_1608Metric, symbol Device:R
- added RED2: RED, LED_SMD:LED_0805_2012Metric, symbol Device:LED
- added SW1: SW_DIP_x01, Button_Switch_SMD:SW_SPDT_PCM12, symbol Switch:SW_SPDT
- added TP1, TP2: Conn_01x01_Female, Connector_PinHeader_2.54mm:PinHeader_1x01_P2.54mm_Vertical, symbol Connector_Generic:Conn_01x01
- added U1: ATGM336H-5N31, KICAD_Footprints:ATGM336H-5N, symbol Connector_Generic:Conn_02x09_Counter_Clockwise
- added U2: LM75B, Package_SO:MSOP-8_3x3mm_P0.65mm, symbol Sensor_Temperature:LM75B
- added U6: DW01, Package_TO_SOT_SMD:SOT-23-6, symbol dw01:DW01
- added U7: TP4056, Package_SO:SOIC-8-1EP_3.9x4.9mm_P1.27mm_EP2.29x3mm_ThermalVias, symbol tp4056:TP4056
- added U8: FS8205A, Package_TO_SOT_SMD:SOT-23-6, symbol fs8205:FS8205A
- R22: renamed from R13; value 10K -> 5K1; LCSC C25804 -> C23186
- S1: value 1 -> PB22; Field5 (none) -> Q 1
- S10: renamed from S15; value R -> PB22; Field5 (none) -> F $
- S11: renamed from S16; value T -> PB22; Field5 (none) -> G %
- S12: renamed from S17; value Y -> PB22; Field5 (none) -> H +
- S13: renamed from S23; value A -> PB22; Field5 (none) -> ALT
- S14: renamed from S24; value S -> PB22; Field5 (none) -> Z <
- S15: renamed from S25; value D -> PB22; Field5 (none) -> X >
- S16: renamed from S26; value F -> PB22; Field5 (none) -> C ?
- S17: renamed from S27; value G -> PB22; Field5 (none) -> V /
- S18: renamed from S28; value H -> PB22; Field5 (none) -> B "
- S19: renamed from S34; value Z -> PB22; Field5 (none) -> ? ?
- S2: value 2 -> PB22; Field5 (none) -> W 2
- S20: renamed from S35; value X -> PB22; Field5 (none) -> ? ?
- S21: renamed from S36; value C -> PB22; Field5 (none) -> ? ?
- S22: renamed from S37; value V -> PB22; Field5 (none) -> ? ?
- S23: renamed from S38; value B -> PB22; Field5 (none) -> ? ?
- S24: renamed from S39; value N -> PB22; Field5 (none) -> ? ?
- S25: renamed from S8; value 8 -> PB22; Field5 (none) -> I 8
- S26: renamed from S9; value 9 -> PB22; Field5 (none) -> O 9
- S27: renamed from S10; value 0 -> PB22; Field5 (none) -> P 0
- S28: renamed from S30; value K -> PB22; Field5 (none) -> M :
- S29: renamed from S31; value L -> PB22; Field5 (none) -> SP
- S3: value 3 -> PB22; Field5 (none) -> E 3
- S30: renamed from S32; value ^ -> PB22; Field5 (none) -> ENT
- S31: renamed from S19; value I -> PB22; Field5 (none) -> K
- S32: renamed from S20; value O -> PB22; Field5 (none) -> L -
- S33: renamed from S21; value P -> PB22; Field5 (none) -> DEL <--
- S34: renamed from S41; value . -> PB22; Field5 (none) -> ? ?
- S35: renamed from S42; value < -> PB22; Field5 (none) -> ? ?
- S36: renamed from S43; value V -> PB22; Field5 (none) -> ? ?
- S4: value 4 -> PB22; Field5 (none) -> R 4
- S5: value 5 -> PB22; Field5 (none) -> T 5
- S6: value 6 -> PB22; Field5 (none) -> Y 6
- S7: renamed from S12; value Q -> PB22; Field5 (none) -> A !
- S8: renamed from S13; value W -> PB22; Field5 (none) -> S &
- S9: renamed from S14; value E -> PB22; Field5 (none) -> D #
- renumbered C6 to C10, C7 to C11, C8 to C12, C9 to C13, C10 to C14, C11 to C15, C13 to C16, C12 to C17, C14 to C18, C15 to C19, C1 to C2, C16 to C20, C18 to C21, C19 to C22, C20 to C23, C21 to C24, C22 to C25, C23 to C26, C2 to C3, C5 to C4, C3 to C5, C4 to C7, D1 to D2, D2 to D3, D3 to D4, JP1 to J2, J1 to J4, J2 to J5, L1 to L2, Q1 to Q2, Q2 to Q3, R9 to R18, R10 to R19, R11 to R20, R12 to R21, R7 to R4, R8 to R5, R4 to R6, R5 to R7, R6 to R8, J3 to TP3, U5 to U10, U6 to U11, U7 to U12, U8 to U13, U9 to U14, U10 to U15, U11 to U16, U12 to U17, U13 to U18, U14 to U19, U15 to U20, U1 to U3, U3 to U4, U2 to U5, U4 to U9
Connections:
- net +3.3V: now also C1.1, SW1.3 (C), U1.6 (Pin_6), U2.8 (+Vs)
- net COL01: now also S25.2, S31.2
- net COL02: now also S26.2, S32.2
- net COL03: now also S27.2, S33.2
- net COL04: now also S28.2, S34.2
- net COL05: now also S29.2, S35.2
- net COL06: now also S30.2, S36.2
- net GND: now also AE1.2 (Shield), C1.2, C8.2, C9.2, J1.2 (Pin_2), J3.1 (Pin_1), R10.1, R11.1, R13.2, R16.2, U1.1 (Pin_1), U1.10 (Pin_10), U1.12 (Pin_12), U2.4 (GND), U2.5 (A2), U2.6 (A1), U2.7 (A0), U7.1 (TEMP), U7.3 (GND), U8.3 (S2); no longer BT1.2 (-), J4.2 (Pin_2)
- net LORA_CS: no longer U4.37 (U0TXD/GPIO43/CLK_OUT1)
- net LORA_SCK: no longer U4.36 (U0RXD/GPIO44/CLK_OUT2)
- net ROW01: no longer S25.1, S26.1, S27.1
- net ROW02: no longer S31.1, S32.1, S33.1
- net ROW03: no longer S28.1, S29.1, S30.1
- net ROW04: no longer S34.1, S35.1, S36.1
- net COL07: no longer names the net of U4.17 (GPIO9/TOUCH9/ADC1_CH8/FSPIHD/SUBSPIHD)
- removed net COL08: S25.2, S28.2, S31.2, S34.2, U4.18 (GPIO10/TOUCH10/ADC1_CH9/FSPICS0/FSPIIO4/SUBSPICS0)
- removed net COL09: S26.2, S29.2, S32.2, S35.2, U4.19 (GPIO11/TOUCH11/ADC2_CH0/FSPICS0/FSPIIO4/SUBSPICS0)
- removed net COL10: S27.2, S30.2, S33.2, S36.2, U4.20 (GPIO12/TOUCH11/ADC2_CH0/FSPICS0/FSPIIO4/SUBSPICS0)
- net COL11: no longer names the net of U4.21 (GPIO13/TOUCH13/ADC2_CH2/FSPIQ/FSPIIO7/SUBSPIQ)
- net VBAT renamed Vdrive
- net Vdrive: now also Q1.3 (S); no longer BT1.1 (+), J4.1 (Pin_1), U12.3 (VBAT)
- new net: C9.1, D1.2 (A), GRN2.2 (A), J3.2 (Pin_2), RED2.2 (A), U7.4 (VCC), U7.8 (CE), U7.9 (PP)
- new net: R15.2, U7.6 (~{STDBY})
- new net: R14.2, U7.7 (~{CHRG})
- new net: GRN2.1 (K), R15.1
- new net: R11.2, U6.2 (CS)
- new net: C6.1, R9.2, U6.5 (VCC)
- new net: J1.1 (Pin_1), SW1.1 (A)
- new net: SW1.2 (B), U1.8 (Pin_8)
- new net: AE1.1 (A), L1.1, U1.11 (Pin_11)
- new net: R14.1, RED2.1 (K)
- new net: Q1.2 (G), R10.2
- new net: L1.2, U1.14 (Pin_14)
- new net +BATT: BT1.1 (+), C8.1, D1.1 (K), J4.2 (Pin_2), Q1.1 (D), R12.1, R9.1, TP1.1 (Pin_1), U12.3 (VBAT), U7.5 (BAT)
- new net BAT-: BT1.2 (-), C6.2, J4.1 (Pin_1), TP2.1 (Pin_1), U6.6 (GND), U8.1 (S1)
- new net G1: U6.1 (OD), U8.6 (G1)
- new net G2: R17.2, U8.4 (G2)
- new net GPS_RX: U1.3 (Pin_3), U4.37 (U0TXD/GPIO43/CLK_OUT1)
- new net GPS_TX: U1.2 (Pin_2), U4.36 (U0RXD/GPIO44/CLK_OUT2)
- new net I2S_SCL: U2.2 (SCL)
- new net I2S_SDA: U2.1 (SDA)
- new net OC: R17.1, U6.3 (OC)
- new net PROG: R16.1, U7.2 (PROG)
- new net ROW05: S25.1, S26.1, S27.1, S28.1, S29.1, S30.1
- new net ROW06: S31.1, S32.1, S33.1, S34.1, S35.1, S36.1
- new net VBATadc: R12.2, R13.1
- no-connect marks 19 -> 32
Other:
- note added: "Ceramic Cap."
- note added: "GPS"
- note added: "SOLAR + PANEL -"
- note added: "SOLAR 18650 BATTERY CHARGER solar notes https://youtu.be/37kGva3NW8w 5V panel, should provide up to 300ma at about 3.3V. https://www.digikey.com/en/products/detail/anysolar-ltd/SM531K08L/9990469"
- note added: "Temp sensor"
- note added: "USB 18650 BATTERY CHARGER"
- note added: "set charge current 10k = 130 ma"
- note removed: "18650 BATTERY CHARGER"
- moved on the sheet: BT1, C17, C2, C21, C3, C4, J2, J4, J5, Q3, R3, R4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

Commit message: DRAFT laying down copper now, many traces still need to be installed. Checked in for archival purposes.
Parts:
- removed AE1: Antenna_Shield, Connector_Coaxial:U.FL_Hirose_U.FL-R-SMT-1_Vertical, symbol Device:Antenna_Shield
- removed GRN2: GRN, LED_SMD:LED_0805_2012Metric, symbol Device:LED
- removed RED2: RED, LED_SMD:LED_0805_2012Metric, symbol Device:LED
- added AE1: Antenna, KICAD_Footprints:KH-GPS181804-WY, symbol Device:Antenna
- added AE2: Conn_Coaxial, Connector_Coaxial:U.FL_Hirose_U.FL-R-SMT-1_Vertical, symbol Connector:Conn_Coaxial
- added C27: 1u, Capacitor_SMD:C_0603_1608Metric, symbol Device:C_Small
- added C28: 4.7uF, Capacitor_SMD:C_0603_1608Metric, symbol Device:C
- added C29: 220n, Capacitor_SMD:C_0603_1608Metric, symbol Device:C
- added C30: 1n, Capacitor_SMD:C_0603_1608Metric, symbol Device:C
- added C31: 1.2p, Capacitor_SMD:C_0603_1608Metric, symbol Device:C
- added C32: 6.8p, Capacitor_SMD:C_0603_1608Metric, symbol Device:C
- added D5: MBR0530, Diode_SMD:D_SOD-123, symbol Diode:MBR0530
- added FL1: TA1661A, KICAD_Footprints:TA1661A, symbol KICAD_ta1661a:TA1661A
- added J5, J6: CONN_01, Connector_Wire:SolderWirePad_1x01_SMD_5x10mm, symbol Connector_Generic:Conn_01x01
- added L3: 6.2nH, Inductor_SMD:L_0603_1608Metric, symbol Device:L
- added R23: 10K, Resistor_SMD:R_0603_1608Metric, symbol Device:R
- added U21: QMC5883L, Package_LGA:LGA-16_3x3mm_P0.5mm, symbol KICAD_qmc5883l:QMC5883L
- added U22: BGU8019, KICAD_Footprints:XSON6, symbol KICAD_bgu8019:BGU8019
- R12, R13: LCSC (none) -> C23162
- R14, R15: value 1K -> 10K; LCSC C21190 -> C25804
- R9: LCSC (none) -> C4184
- S10: renamed from S22; Field5 ? ? -> P 0
- S12: renamed from S24; Field5 ? ? -> DEL
- S14: renamed from S8; Field5 S & -> S @
- S19: renamed from S25; Field5 I 8 -> J &
- S20: renamed from S26; Field5 O 9 -> K
- S21: renamed from S27; Field5 P 0 -> L -
- S22: renamed from S28; Field5 M : -> ?
- S23: renamed from S29; Field5 SP -> ^
- S31: Field5 K -> N ;
- S32: Field5 L - -> M :
- S33: Field5 DEL <-- -> SPC
- S34: Field5 ? ? -> <
- S35: Field5 ? ? -> V
- S36: Field5 ? ? -> >
- S7: renamed from S19; Field5 ? ? -> U 7
- S8: renamed from S20; Field5 ? ? -> I 8
- S9: renamed from S21; Field5 ? ? -> O 9
- TP2: renamed from TP1; value Conn_01x01_Female -> CONN_01; LCSC (none) -> DNP
- TP3: renamed from TP2; value Conn_01x01_Female -> CONN_01; LCSC (none) -> DNP
- U3: footprint KICAD_Footprints:USB-C_SMD-TYPE-C-31-M-12 -> tp4056:USB-C_SMD-TYPE-C-31-M-12; symbol USB:tp4056_KoreanHropartsElecTYPE-C-31-M-12 -> KICAD_USB:tp4056_KoreanHropartsElecTYPE-C-31-M-12
- U4: footprint KICAD_Footprints:ESP32-S3-WROOM-1 -> Espressif:ESP32-S3-WROOM-1; symbol ESP32:Espressif_ESP32-S3-WROOM-1 -> KICAD_ESP32:Espressif_ESP32-S3-WROOM-1
- U5: symbol armachat-eagle-import:RFM69HCW -> KICAD_rfm69hcw:RFM69HCW
- U6: symbol dw01:DW01 -> KICAD_dw01:DW01
- U7: symbol tp4056:TP4056 -> KICAD_tp4056:TP4056
- U8: symbol fs8205:FS8205A -> KICAD_fs8205a:FS8205A
- renumbered J3 to J2, J4 to J3, J5 to J4, R3 to R1, R4 to R2, R5 to R3, R6 to R4, R1 to R5, R2 to R6, S23 to S11, S7 to S13, S9 to S15, S10 to S16, S11 to S17, S12 to S18, S30 to S24, S13 to S25, S14 to S26, S15 to S27, S16 to S28, S17 to S29, S18 to S30, J2 to TP1, TP3 to TP4
Connections:
- net +3.3V: now also SW1.1 (A), C27.1, D5.2 (A), U21.13 (VDDIO), U21.2 (VDD), U21.4 (S1); no longer SW1.3 (C), U5.5P (VDD)
- net +BATT: now also J5.1 (Pin_1)
- net BAT-: now also J6.1 (Pin_1)
- net COL01: now also S12.2, S24.2, S36.2; no longer S19.2, S31.2, S7.2
- net COL02: now also S11.2, S23.2, S35.2; no longer S20.2, S32.2, S8.2
- net COL03: now also S10.2, S22.2, S34.2; no longer S21.2, S33.2, S9.2
- net COL04: now also S21.2, S33.2, S9.2; no longer S10.2, S22.2, S34.2
- net COL05: now also S20.2, S32.2, S8.2; no longer S11.2, S23.2, S35.2
- net COL06: now also S19.2, S31.2, S7.2; no longer S12.2, S24.2, S36.2
- net DIO1: no longer U5.7P (DIO1)
- net DIO2: no longer U5.8P (DIO2)
- net DIO3: no longer U5.3P (DIO3)
- net DIO4: no longer U5.4P (DIO4)
- net DIO5: no longer U5.15P (DIO5)
- net GND: now also AE2.2 (Ext), C27.2, C28.1, C30.2, C32.2, FL1.2, FL1.3, FL1.4, R23.1, U21.11 (GND), U21.9 (GND), U22.1 (GND), U22.2 (VCC), U22.4 (EP); no longer U5.16P (GND@3), U5.2P (GND@1), U5.9P (GND@2)
- net I2S_SCL: now also U21.1 (SCL)
- net I2S_SDA: now also U21.16 (SDA)
- net LORA_CS: no longer U5.13P (NSS)
- net LORA_IRQ: no longer U5.6P (DIO0)
- net LORA_MISO: no longer U5.10P (MISO)
- net LORA_MOSI: no longer U5.11P (MOSI)
- net LORA_RST: no longer U5.14P (RESET)
- net LORA_SCK: no longer U5.12P (SCK)
- net at C9.1, D1.2 (A), J2.2 (Pin_2)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: now also R14.1, R15.1; no longer U7.9 (PP)
- net SOLAR_STDBY: now reaches R15.2, U7.6 (~{STDBY})
- net SOLAR_CHRG: now reaches R14.2, U7.7 (~{CHRG})
- net at TP1.1 (Pin_1), U5.1 (ANT), X1.1 (In): no longer U5.1P (ANT)
- net at J1.1 (Pin_1): now also SW1.3 (C); no longer SW1.1 (A)
- net RF_OUT: now reaches L1.1, U1.11 (Pin_11)
- net RF_OUT: now also AE2.1 (In), FL1.5
- new net: C30.1, D5.1 (K), R23.2, U22.2 (VCC), U22.6 (VENABLE)
- new net: C32.1, L3.1
- new net: C31.2, L3.2, U22.5 (RFIN)
- new net: AE1.1 (A), C31.1
- new net C1: C28.2, U21.10 (C1)
- new net COMP_DATA_READY: U21.15 (DRDY)
- new net RF_IN: FL1.1, U22.3 (RFOUT)
- new net SETC: C29.1, U21.12 (SETC)
- new net SETP: C29.2, U21.8 (SETP)
- no-connect marks 32 -> 33
Other:
- note added: "BGU8019 V range is 1.5 to 3.1V so diode drop 3.3V."
- note added: "COMPASS"
- note added: "Ref https://youtu.be/-fuOCj-e7sM"
- note added: "TEMPERATURE"
- note added: "optional GPS battery, or power off GPS."
- note added: "optional extranl battery"
- note added: "optional extranl speaker"
- note removed: "Temp sensor"
- moved on the sheet: C1, GRN1, J1, L1, R14, R15, R5, R6, RED1, S10, S11, S12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

Commit message: DRAFT Almost ready for review again. Checking in for archival purposes.
Parts:
- added TP10, TP11, TP12, TP13, TP14, TP15, TP16, TP17, TP18, TP19, TP20, TP21, TP22, TP23, TP24, TP25, TP26, TP27, TP28, TP29, TP30, TP31, TP32, TP33, TP34, TP35, TP36, TP37, TP5, TP6, TP7, TP8, TP9: CONN_01, KICAD_Footprints:TST_x01_P2.54mm_Vertical, symbol Connector_Generic:Conn_01x01
- TP1, TP2, TP3, TP4: footprint Connector_PinHeader_2.54mm:PinHeader_1x01_P2.54mm_Vertical -> KICAD_Footprints:TST_x01_P2.54mm_Vertical
- U3: footprint tp4056:USB-C_SMD-TYPE-C-31-M-12 -> KICAD_Footprints:USB-C_SMD-TYPE-C-31-M-12
- U4: footprint Espressif:ESP32-S3-WROOM-1 -> KICAD_Footprints:ESP32-S3-WROOM-1
Connections:
- net IO06 is gone; now on net COL01: U4.6 (GPIO6/TOUCH6/ADC1_CH5)
- net IO07 is gone; now on net COL02: U4.7 (GPIO7/TOUCH7/ADC1_CH6)
- net IO15 is gone; now on net COL03: U4.8 (GPIO15/U0RTS/ADC2_CH4/XTAL_32K_P)
- net COL01: now also TP27.1 (Pin_1); no longer U4.9 (GPIO16/U0CTS/ADC2_CH5/XTAL_32K_NH5)
- net COL02: now also TP28.1 (Pin_1); no longer U4.10 (GPIO17/U1TXD/ADC2_CH6)
- net COL03: now also TP33.1 (Pin_1); no longer U4.11 (GPIO18/U1RXD/ADC2_CH7/CLK_OUT3)
- net COL04: now also U4.9 (GPIO16/U0CTS/ADC2_CH5/XTAL_32K_NH5), TP34.1 (Pin_1); no longer U4.12 (GPIO8/TOUCH8/ADC1_CH7/SUBSPICS1)
- net COL05: now also U4.10 (GPIO17/U1TXD/ADC2_CH6), TP35.1 (Pin_1); no longer U4.15 (GPIO3/TOUCH3/ADC1_CH2)
- net COL06: now also U4.11 (GPIO18/U1RXD/ADC2_CH7/CLK_OUT3), TP36.1 (Pin_1); no longer U4.16 (GPIO46)
- net COMP_DATA_READY: now also U4.26 (GPIO45), TP10.1 (Pin_1)
- net DN: no longer U3.B7 (DN2)
- net DP: no longer U3.B6 (DP2)
- net EPD_BUSY: now also U4.25 (GPIO48/SPICLK_N/SUBSPICLK_N_DIFF), TP11.1 (Pin_1); no longer U4.32 (MTCK/GPIO39/CLK_OUT3/SUBSPICS1)
- net EPD_CLK: now also U4.21 (GPIO13/TOUCH13/ADC2_CH2/FSPIQ/FSPIIO7/SUBSPIQ), TP17.1 (Pin_1); no longer U4.28 (SPIIO6/GPIO35/FSPID/SUBSPID)
- net EPD_CS: now also U4.22 (GPIO14/TOUCH14/ADC2_CH3/FSPIWP/FSPIDQS/SUBSPIWP), TP19.1 (Pin_1); no longer U4.29 (SPIIO7/GPIO36/FSPICLK/SUBSPICLK)
- net EPD_DC: now also U4.23 (GPIO21), TP9.1 (Pin_1); no longer U4.30 (SPIDQS/GPIO37/FSPIQ/SUBSPIQ)
- net EPD_MOSI: now also U4.20 (GPIO12/TOUCH11/ADC2_CH0/FSPICS0/FSPIIO4/SUBSPICS0), TP15.1 (Pin_1); no longer U4.26 (GPIO45)
- net EPD_RST: now also U4.24 (GPIO47/SPICLK_P/SUBSPICLK_P_DIFF), TP12.1 (Pin_1); no longer U4.31 (GPIO38/FSPIWP/SUBSPIWP)
- net GPS_RX: now also TP6.1 (Pin_1)
- net GPS_TX: now also TP8.1 (Pin_1)
- net I2S_SCL: now also U4.34 (MTDI/GPIO41/CLK_OUT1), TP23.1 (Pin_1)
- net I2S_SDA: now also U4.35 (MTMS/GPIO42), TP22.1 (Pin_1)
- net LORA_CS: now also U4.31 (GPIO38/FSPIWP/SUBSPIWP), TP18.1 (Pin_1)
- net LORA_IRQ: now also U4.32 (MTCK/GPIO39/CLK_OUT3/SUBSPICS1), TP20.1 (Pin_1); no longer U4.39 (GPIO1/TOUCH1/ADC1_CH0)
- net LORA_MISO: now also U4.28 (SPIIO6/GPIO35/FSPID/SUBSPID), TP13.1 (Pin_1); no longer U4.34 (MTDI/GPIO41/CLK_OUT1)
- net LORA_MOSI: now also U4.29 (SPIIO7/GPIO36/FSPICLK/SUBSPICLK), TP14.1 (Pin_1); no longer U4.35 (MTMS/GPIO42)
- net LORA_RST: now also U4.33 (MTDO/GPIO40/CLK_OUT2), TP21.1 (Pin_1); no longer U4.38 (GPIO2/TOUCH2/ADC1_CH1)
- net LORA_SCK: now also U4.30 (SPIDQS/GPIO37/FSPIQ/SUBSPIQ), TP16.1 (Pin_1)
- net ROW01: now also U4.12 (GPIO8/TOUCH8/ADC1_CH7/SUBSPICS1), TP29.1 (Pin_1); no longer U4.22 (GPIO14/TOUCH14/ADC2_CH3/FSPIWP/FSPIDQS/SUBSPIWP)
- net ROW02: now also U4.15 (GPIO3/TOUCH3/ADC1_CH2), TP24.1 (Pin_1); no longer U4.23 (GPIO21)
- net ROW03: now also U4.16 (GPIO46), TP37.1 (Pin_1); no longer U4.24 (GPIO47/SPICLK_P/SUBSPICLK_P_DIFF)
- net ROW04: now also U4.17 (GPIO9/TOUCH9/ADC1_CH8/FSPIHD/SUBSPIHD), TP30.1 (Pin_1); no longer U4.25 (GPIO48/SPICLK_N/SUBSPICLK_N_DIFF)
- net ROW05: now also U4.18 (GPIO10/TOUCH10/ADC1_CH9/FSPICS0/FSPIIO4/SUBSPICS0), TP31.1 (Pin_1)
- net ROW06: now also U4.19 (GPIO11/TOUCH11/ADC2_CH0/FSPICS0/FSPIIO4/SUBSPICS0), TP32.1 (Pin_1)
- net RXLED: now also TP26.1 (Pin_1)
- net SPEAKPWM: now also U4.38 (GPIO2/TOUCH2/ADC1_CH1), TP7.1 (Pin_1); no longer U4.33 (MTDO/GPIO40/CLK_OUT2)
- net TXLED: now also TP25.1 (Pin_1)
- net VBATadc: now also U4.39 (GPIO1/TOUCH1/ADC1_CH0), TP5.1 (Pin_1)
- net VBUS: no longer U3.B4 (VBUS)
- net USBstat: now reaches R21.2, U12.1 (STAT)
- net at C9.1, D1.2 (A), J2.2 (Pin_2)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: now also U7.9 (PP)
- no-connect marks 33 -> 32
Other:
- note added: "Ref https://youtu.be/-fuOCj-e7sM I2C address is 0D: 0001101 QMC5883L has a built-in temperature sensor"
- note removed: "Ref https://youtu.be/-fuOCj-e7sM"

Commit message: Ready for review.
Parts:
- renumbered C2 to C1, C26 to C10, C21 to C11, C17 to C12, C3 to C13, C31 to C14, C14 to C15, C32 to C16, C30 to C17, C11 to C18, C27 to C19, C9 to C2, C7 to C20, C10 to C21, C13 to C22, C16 to C23, C19 to C24, C5 to C25, C12 to C26, C15 to C27, C18 to C28, C20 to C29, C4 to C3, C28 to C30, C29 to C31, C1 to C32, C22 to C4, C8 to C5, C23 to C6, C24 to C7, C6 to C8, C25 to C9, D5 to D2, D2 to D3, D3 to D4, D4 to D5, J2 to J1, J5 to J2, J6 to J3, J3 to J4, J4 to J5, J1 to J6, L3 to L1, L1 to L3, Q3 to Q2, Q2 to Q3, R2 to R1, R17 to R10, R9 to R11, R4 to R13, R7 to R14, R13 to R15, R10 to R16, R1 to R17, R8 to R18, R23 to R19, R3 to R2, R18 to R20, R5 to R21, R6 to R22, R19 to R23, R14 to R3, R15 to R4, R22 to R5, R21 to R6, R16 to R7, R11 to R8, R20 to R9, S4 to S10, S16 to S11, S28 to S12, S5 to S13, S17 to S14, S29 to S15, S6 to S16, S18 to S17, S30 to S18, S7 to S19, S13 to S2, S19 to S20, S31 to S21, S8 to S22, S20 to S23, S32 to S24, S9 to S25, S21 to S26, S33 to S27, S10 to S28, S22 to S29, S25 to S3, S34 to S30, S11 to S31, S23 to S32, S35 to S33, S12 to S34, S24 to S35, S2 to S4, S14 to S5, S26 to S6, S3 to S7, S15 to S8, S27 to S9, TP5 to TP1, TP31 to TP10, TP32 to TP11, TP15 to TP12, TP17 to TP13, TP19 to TP14, TP33 to TP15, TP34 to TP16, TP35 to TP17, TP36 to TP18, TP2 to TP19, TP7 to TP2, TP3 to TP20, TP6 to TP21, TP8 to TP22, TP9 to TP23, TP10 to TP24, TP37 to TP25, TP11 to TP26, TP12 to TP27, TP13 to TP28, TP14 to TP29, TP24 to TP3, TP16 to TP30, TP18 to TP31, TP20 to TP32, TP21 to TP33, TP23 to TP34, TP22 to TP35, TP4 to TP36, TP1 to TP37, TP25 to TP4, TP26 to TP5, TP27 to TP6, TP28 to TP7, TP29 to TP8, TP30 to TP9, U12 to U1, U13 to U10, U17 to U11, U14 to U12, U18 to U13, U15 to U14, U19 to U15, U20 to U17, U22 to U18, U2 to U19, U7 to U2, U1 to U20, U10 to U22, U4 to U3, U8 to U4, U6 to U5, U11 to U6, U5 to U7, U3 to U8

Commit message: Some corrections to align with JLCPCB verification, added I2C memory chip.
Parts:
- added C14: 100n, Capacitor_SMD:C_0603_1608Metric, symbol Device:C
- added SC1: Solar_Cell, symbol Device:Solar_Cell
- added U16: MB85RC64, Package_SO:SOP-8_3.9x4.9mm_P1.27mm, symbol Memory_EEPROM:24LC00
- C15: renamed from C14; LCSC (none) -> C281768
- C17: renamed from C16; LCSC (none) -> C1679
- C18: renamed from C17; LCSC (none) -> C100040
- FL1: LCSC (none) -> C2961690
- L1: LCSC (none) -> C98083
- U19: renamed from U18; LCSC (none) -> C3190009
- U22: renamed from U21; LCSC (none) -> C976032
- U4: footprint Package_TO_SOT_SMD:SOT-23-6 -> Package_SO:TSSOP-8_4.4x3mm_P0.65mm
- renumbered C15 to C16, C18 to C19, C19 to C20, C20 to C21, C21 to C22, C22 to C23, C23 to C24, C24 to C25, C25 to C26, C26 to C27, C27 to C28, C28 to C29, C29 to C30, C30 to C31, C31 to C32, C32 to C33, U16 to U17, U17 to U18, U19 to U20, U20 to U21, U22 to U23
Connections:
- net +3.3V: now also C14.2, U16.1 (A0), U16.7 (WP), U16.8 (VCC)
- net BAT-: now also U4.6 (S2), U4.7 (S2); no longer U4.1 (S1)
- net G1: now also U4.5 (G2); no longer U4.6 (G1)
- net GND: now also U4.2 (S1), C14.1, U16.2 (A1), U16.3 (A2), U16.4 (GND)
- net I2S_SCL: now also U16.6 (SCL)
- net I2S_SDA: now also U16.5 (SDA)
- no-connect marks 32 -> 34
Other:
- note added: "MEMORY"
