File: ESP32chat.kicad_sch (KiCad schematic)
At the start: 181 parts, among them J1 CONN_021X02_NO_SILK, J2 CONN_01, J3 CONN_01, J4 CONN_021X02_NO_SILK, J5 CONN_021X02_NO_SILK, J6 CONN_021X02_NO_SILK, Q1 Q_PMOS_DGS, Q2 BSS123, Q3 Si1308, SW1 SW_DIP_x01, U1 MCP73831T-2ACI/OT, U10 MOUNTINGHOLE2.0, U11 MOUNTINGHOLE2.0, U12 MOUNTINGHOLE2.0, U13 MOUNTINGHOLE2.0, U14 MOUNTINGHOLE2.0, U15 MOUNTINGHOLE2.0, U16 MB85RC64, U17 MOUNTINGHOLE2.0, U18 MOUNTINGHOLE2.0, U19 BGU8019, U2 TP4056, U20 LM75B, U21 ATGM336H-5N31, U22 QMC5883L, U23 FPCConn, U3 ESP32, U4 FS8205A, U5 DW01, U6 RT9013, U7 RFM69HCW, U8 tp4056_KoreanHropartsElecTYPE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, U9 BUZZER, X1 uFL

Commit message: Added SD memory, Added 2nd USB for 232 initial circuit python programming
Parts:
- removed C14: 100n, Capacitor_SMD:C_0603_1608Metric, symbol Device:C
- removed U16: MB85RC64, Package_SO:SOP-8_3.9x4.9mm_P1.27mm, symbol Memory_EEPROM:24LC00
- added C11, C13, C21, C33, C37: 100n, Capacitor_SMD:C_0603_1608Metric, symbol Device:C
- added C38: 1u, Capacitor_SMD:C_0603_1608Metric, symbol Device:C_Small
- added J2, J3: CONN_021X02_NO_SILK, Connector_PinHeader_2.54mm:PinHeader_1x02_P2.54mm_Vertical, symbol Connector_Generic:Conn_01x02
- added J8: Micro_SD_Card_Det, KICAD_Footprints:microSD_HC_Molex_104031-0811_Modified_for_JLCPCB, symbol Connector:Micro_SD_Card_Det
- added Q4, Q5: Q_NPN_BEC, KICAD_Footprints:SOT-23_Modified_for_JLCPCB, symbol Device:Q_NPN_BEC
- added R12, R14, R43, R44: 10K, Resistor_SMD:R_0603_1608Metric, symbol Device:R
- added R20, R21, R25, R26, R27, R28, R29, R30, R31, R32, R33, R36, R37, R39, R40, R41, R42: 0R, Resistor_SMD:R_0603_1608Metric, symbol Device:R
- added R45: 10K DNP, Resistor_SMD:R_0603_1608Metric, symbol Device:R
- added R46: 1K, Resistor_SMD:R_0603_1608Metric, symbol armachat-eagle-import:RESISTOR_0603_NOOUT
- added R47, R48: 22K1, Resistor_SMD:R_0603_1608Metric, symbol Device:R
- added R49, R51, R52: 0R, Resistor_SMD:R_2010_5025Metric, symbol Device:R
- added R50: 5K1, Resistor_SMD:R_0603_1608Metric, symbol Device:R
- added R53: 1K, Resistor_SMD:R_0603_1608Metric, symbol Device:R
- added SW2: SW_Push_DPDT, Button_Switch_THT:SW_E-Switch_EG1271_DPDT, symbol Switch:SW_Push_DPDT
- added TP38, TP39, TP40, TP41, TP42, TP43, TP44, TP45, TP46: CONN_01, KICAD_Footprints:TST_x01_P2.54mm_Vertical, symbol Connector_Generic:Conn_01x01
- added U24: CP2102N-Axx-xQFN28, Package_DFN_QFN:QFN-28-1EP_5x5mm_P0.5mm_EP3.35x3.35mm, symbol Interface_USB:CP2102N-Axx-xQFN28
- added U25: tp4056_KoreanHropartsElecTYPE-C-31-M-12, KICAD_Footprints:USB-C_SMD-TYPE-C-31-M-12, symbol KICAD_USB:tp4056_KoreanHropartsElecTYPE-C-31-M-12
- added U9: PCA9555PW, KICAD_Footprints:TSSOP-24_4.4x7.8mm_P0.65mm_Modified_for_JLCPCB, symbol Interface_Expansion:PCA9555PW
- Q1, Q2: footprint Package_TO_SOT_SMD:SOT-23 -> KICAD_Footprints:SOT-23_Modified_for_JLCPCB
- Q3: footprint Package_TO_SOT_SMD:SOT-323_SC-70 -> KICAD_Footprints:SOT-323_SC-70_Modified_for_JLCPCB
- U1: footprint Package_TO_SOT_SMD:SOT-23-5 -> KICAD_Footprints:SOT-23-5_Modified_for_JLCPCB-5
- U2: footprint Package_SO:SOIC-8-1EP_3.9x4.9mm_P1.27mm_EP2.29x3mm_ThermalVias -> KICAD_Footprints:SOIC-8-1EP_3.9x4.9mm_P1.27mm_EP2.29x3mm_Therm_Modified_for_JLCPCB
- U20: footprint Package_SO:MSOP-8_3x3mm_P0.65mm -> KICAD_Footprints:MSOP-8_3x3mm_P0.65mm_Modified_for_JLCPCB
- U4: footprint Package_SO:TSSOP-8_4.4x3mm_P0.65mm -> KICAD_Footprints:TSSOP-8_4.4x3mm_P0.65mm_Modified_for_JLCPCB
- U5: footprint Package_TO_SOT_SMD:SOT-23-6 -> KICAD_Footprints:SOT-23-6_Modified_for_JLCPCB
- U6: footprint Package_TO_SOT_SMD:SOT-23-5 -> KICAD_Footprints:SOT-23-5_Modified_for_JLCPCB
- X1: footprint Connector_Coaxial:SMA_Molex_73251-2200_Horizontal -> KICAD_Footprints:SMA_Molex_73251-2200_Horizontal_Modified_for_JLCPCB
- renumbered C13 to C12, C15 to C14, C16 to C15, C17 to C16, C11 to C17, C12 to C19, C19 to C20, C20 to C22, C21 to C23, C22 to C24, C23 to C25, C24 to C26, C25 to C27, C26 to C28, C27 to C29, C28 to C30, C29 to C31, C30 to C32, C31 to C34, C32 to C35, C33 to C36, J2 to J4, J3 to J5, J4 to J6, J5 to J7, J6 to J9, R12 to R13, R13 to R15, R14 to R16, R15 to R17, R16 to R18, R17 to R19, R18 to R22, R21 to R23, R22 to R24, R19 to R34, R20 to R35, R23 to R38, TP37 to TP36, TP36 to TP37, U17 to U16, U18 to U17, U19 to U18, U9 to U19
Connections:
- net +3.3V: now also C11.2, C13.2, C21.2, C33.2, C37.2, J8.4 (VDD), R12.2, R14.2, R46.1, U24.6 (VDD), U24.7 (VREGIN), U9.2 (A1), U9.24 (VDD)
- net COMP_DATA_READY: now also U9.4 (IO0_0); no longer TP24.1 (Pin_1), U3.26 (GPIO45)
- net GND: now also C11.1, C13.1, C21.1, C33.1, C37.1, C38.2, J2.1 (Pin_1), J3.1 (Pin_1), J8.11 (SHIELD), J8.6 (VSS), R45.1, R47.1, R50.1, R53.2, U24.29 (GND), U24.3 (GND), U25.0, U25.A1 (GND), U25.A12 (GND), U25.B1 (GND), U25.B12 (GND), U9.12 (VSS), U9.21 (A0), U9.3 (A2)
- net GPS_RX: now also R41.1, SW2.1 (A); no longer TP21.1 (Pin_1), U21.3 (Pin_3), U3.37 (U0TXD/GPIO43/CLK_OUT1)
- net GPS_TX: now also R42.1, SW2.4 (A); no longer TP22.1 (Pin_1), U21.2 (Pin_2), U3.36 (U0RXD/GPIO44/CLK_OUT2)
- net I2S_SCL: now also R12.1, R20.2, R37.2; no longer U20.2 (SCL)
- net I2S_SDA: now also R14.1, R21.2, R36.2; no longer U20.1 (SDA)
- net SOLAR_CHRG: now also U9.18 (IO1_5)
- net SOLAR_STDBY: now also U9.17 (IO1_4)
- net SPEAKPWM: now also R25.2; no longer C17.2, Q2.1 (G), TP37.1 (Pin_1)
- net USBstat: now also U9.16 (IO1_3)
- net ESP32_BOOT: now reaches R2.2, U3.27 (GPIO0/BOOT)
- net ESP32_BOOT: now also J2.2 (Pin_2), R39.2
- net EN renamed ESP32_EN
- net ESP32_EN: now also J3.2 (Pin_2), R40.2
- net LORA_MISO renamed HS_MISO
- net HS_MISO: now also R30.1
- net LORA_MOSI renamed HS_MOSI
- net HS_MOSI: now also R28.1
- net LORA_SCK renamed HS_SCK
- net HS_SCK: now also R29.1
- new net: R48.2, R49.2
- new net: Q4.1 (B), R43.2
- new net: Q4.3 (C), R39.1
- new net: Q5.1 (B), R44.2
- new net: Q5.3 (C), R40.1
- new net: R41.2, U21.3 (Pin_3)
- new net: R51.1, U25.A6 (DP1)
- new net: R36.1, U20.1 (SDA)
- new net: R37.1, U20.2 (SCL)
- new net: TP43.1 (Pin_1), U9.6 (IO0_2)
- new net: TP40.1 (Pin_1), U9.19 (IO1_6)
- new net: R46.2, U24.9 (~{RST})
- new net: J8.2 (DAT3/CD), R27.2
- new net: TP45.1 (Pin_1), U9.14 (IO1_1)
- new net: TP46.1 (Pin_1), U9.15 (IO1_2)
- new net: TP41.1 (Pin_1), U9.20 (IO1_7)
- new net: R20.1, U9.22 (SCL)
- new net: R21.1, U9.23 (SDA)
- new net: TP42.1 (Pin_1), U9.5 (IO0_1)
- new net: TP44.1 (Pin_1), U9.7 (IO0_3)
- new net: J8.8 (DAT1), R31.2
- new net: C17.2, Q2.1 (G), R25.1, TP37.1 (Pin_1)
- new net: J8.1 (DAT2), R26.2
- new net: J8.9 (DET_B), R33.2
- new net: R50.2, U25.A5 (CC1)
- new net: R52.1, U25.A7 (DN1)
- new net: R53.1, U25.B5 (CC2)
- new net: J8.10 (DET_A), R32.2
- new net: J8.3 (CMD), R28.2
- new net: J8.5 (CLK), R29.2
- new net: J8.7 (DAT0), R30.2
- new net: R45.2, U24.11 (~{SUSPEND})
- new net: R42.2, U21.2 (Pin_2)
- new net +5VP: R49.1, U25.A4 (VBUS), U25.A9 (VBUS), U25.B9 (VBUS)
- new net DN232: R52.2, U24.5 (D-)
- new net DP232: R51.2, U24.4 (D+)
- new net ESP32_RX: SW2.2 (B), TP21.1 (Pin_1), U3.37 (U0TXD/GPIO43/CLK_OUT1)
- new net ESP32_TX: SW2.5 (B), TP22.1 (Pin_1), U3.36 (U0RXD/GPIO44/CLK_OUT2)
- new net EXPAND_INT: TP24.1 (Pin_1), U3.26 (GPIO45), U9.1 (~{INT})
- new net SDCard_CS: R27.1, U9.8 (IO0_4)
- new net SDCard_Dat1: R31.1, U9.13 (IO1_0)
- new net SDCard_Dat2: R26.1, U9.9 (IO0_5)
- new net SDCard_DetA: R32.1, U9.11 (IO0_7)
- new net SDCard_DetB: R33.1, U9.10 (IO0_6)
- new net USBDTR: Q4.2 (E), R44.1, TP39.1 (Pin_1), U24.28 (~{DTR})
- new net USBRTS: Q5.2 (E), R43.1, TP38.1 (Pin_1), U24.24 (~{RTS})
- new net USB_RX: SW2.3 (C), U24.25 (RXD)
- new net USB_TX: SW2.6 (C), U24.26 (TXD)
- new net VBUS232: C38.1, R47.2, R48.1, U24.8 (VBUS)
- no-connect marks 34 -> 54
Other:
- note added: "Auto program ADD1 ADD2 ADD3 --> DEVICE 0 0 0 TEMPERATURE 0 1 0 EXPANDER COMPAS I2C address is 0D: 0001101"
- note added: "Auto program DTR RTS-->EN IO0 IO2 1 1 1 1 1 0 0 1 1 1 1 0 0 1 1 0 1 1 0 0"
- note added: "I2C EXPANSION IO"
- note added: "LORA RADIO"
- note added: "Perhaps remove this section and replace with the below https://www.adafruit.com/product/5335"
- note added: "SD MEMORY"
- note added: "SPEAKER"
- note added: "USB INITIAL PROGRAMING INTERFACE"
- note added: "optional external battery"
- note added: "optional external speaker"
- note added: "switch would go away if we remove this section"
- note removed: "MEMORY"
- note removed: "Speaker"
- note removed: "optional extranl battery"
- note removed: "optional extranl speaker"
- moved on the sheet: C1, C12, C15, C17, C19, C20, C22, C34, C35, D3, D4, D5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
