File: ESP32chat.kicad_sch (KiCad schematic)
At the start: 233 parts, among them J1 CONN_021X02_NO_SILK, J2 CONN_021X02_NO_SILK, J3 CONN_021X02_NO_SILK, J4 CONN_01, J5 CONN_01, J6 CONN_021X02_NO_SILK, J7 CONN_021X02_NO_SILK, J8 Micro_SD_Card_Det, J9 CONN_021X02_NO_SILK, Q1 Q_PMOS_DGS, Q2 BSS123, Q3 Si1308, Q4 Q_NPN_BEC, Q5 Q_NPN_BEC, SW1 SW_DIP_x01, SW2 SW_Push_DPDT, U1 MCP73831T-2ACI/OT, U10 MOUNTINGHOLE2.0, U11 MOUNTINGHOLE2.0, U12 MOUNTINGHOLE2.0, U13 MOUNTINGHOLE2.0, U14 MOUNTINGHOLE2.0, U15 MOUNTINGHOLE2.0, U16 MOUNTINGHOLE2.0, U17 MOUNTINGHOLE2.0, U18 BGU8019, U19 BUZZER, U2 TP4056, U20 LM75B, U21 ATGM336H-5N31, U22 QMC5883L, U23 FPCConn, U24 CP2102N-Axx-xQFN28, U25 tp4056_KoreanHropartsElecTYPE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, U3 ESP32, U4 FS8205A, U5 DW01, U6 RT9013, U7 RFM69HCW, U8 tp4056_KoreanHropartsElecTYPE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, U9 PCA9555PW, X1 uFL

Commit message: Updated BOM
Parts:
- U3: LCSC C2913199 -> C2913204
Changed lines of the file:
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@@
       (effects (font (size 1.27 1.27)) hide)
     )
-    (property "LCSC" "C2913199" (id 4) (at 109.22 121.285 0)
+    (property "LCSC" "C2913204" (id 4) (at 109.22 121.285 0)
       (effects (font (size 1.27 1.27)) hide)
     )
